Commit message: Testing input arguments for simulation launch. Corrected for arguments that were not well propagated.

File: vizzy_description/plugins/ros.gazebo.xacro (robot description, xacro)
@@ -5,4 +5,7 @@
 -->
 <root xmlns:xacro="http://ros.org/wiki/xacro">
+  <xacro:arg name="odom_topic" default="model/vizzy/odometry"/>
+  <xacro:arg name="odom_frame_id" default="odometry"/>
+  <xacro:arg name="base_frame_id" default="base_footprint"/>
   <!-- Joint States Publisher -->
   <xacro:macro name="joint_state_publisher">
@@ -31,7 +34,7 @@
           <publish_odom_tf>true</publish_odom_tf>
           <publish_wheel_tf>true</publish_wheel_tf>
-          <odom_topic>model/vizzy/odometry</odom_topic>
-          <frame_id>odometry</frame_id>
-          <child_frame_id>base_footprint</child_frame_id>
+          <odom_topic>$(arg odom_topic)</odom_topic>
+          <frame_id>$(arg odom_frame_id)</frame_id>
+          <child_frame_id>$(arg base_frame_id)</child_frame_id>
           <tf_topic>model/vizzy/tf</tf_topic>
       </plugin>

File: vizzy_description/robots/vizzy.urdf.xacro (robot description, xacro)
@@ -6,12 +6,11 @@
 -->
 <robot  name="vizzy" xmlns:xacro="http://ros.org/wiki/xacro" >
-  <!-- Load Yarp plugins for real robot execution -->
   <xacro:arg name="use_yarp" default="false"/>
-  <!-- Load full inertial and collision model or a simplified model -->
   <xacro:arg name="use_full_gazebo_model" default="false"/>
-  <!-- Load a fully detailed hand model with properly modeled links and joints -->
   <xacro:arg name="use_full_hand_model" default="false"/>
-  <!-- Disable laser sensors -->
   <xacro:arg name="disable_laser" default="true"/>
+  <xacro:arg name="odom_topic"         default="/odom" />
+  <xacro:arg name="odom_frame_id"      default="odometry" />
+  <xacro:arg name="base_frame_id"   default="base_footprint" />
   <!-- Includes -->
   <!-- Misc common stuff such as constant definitions -->

File: vizzy_description/urdf/base/base.urdf.xacro (robot description, xacro)
@@ -6,4 +6,5 @@
   <!-- Load full inertial and collision model or a simplified model -->
   <xacro:arg name="use_full_gazebo_model" default="false"/>
+  <xacro:arg name="base_frame_id" default="base_footprint"/>
   <!-- Things that are needed only for Gazebo (not the physical robot).  These include
        sensor and controller plugin specifications -->
@@ -13,11 +14,11 @@
   <xacro:macro name="base" params="name">
     <!-- Root link, on the ground just below the robot origin -->
-    <link name="base_footprint">
+    <link name="$(arg base_frame_id)">
     </link>
-    <joint name="base_footprint_joint" type="fixed">
+    <joint name="$(arg base_frame_id)_joint" type="fixed">
       <origin
         xyz="0.1934543 0.0 0.04"
         rpy="0.0 0.0 ${M_PI}"/>
-      <parent link="base_footprint"/>
+      <parent link="$(arg base_frame_id)"/>
       <child link="base_link"/>
     </joint>

File: vizzy_description/urdf/simple_base/base.gazebo.xacro (robot description, xacro)
@@ -1,4 +1,5 @@
 <?xml version="1.0"?>
 <robot xmlns:xacro="http://ros.org/wiki/xacro">
+  <xacro:arg name="base_frame_id" default="base_footprint"/>
   <xacro:macro name="base_gazebo">
     <gazebo reference="base_link">
@@ -6,5 +7,5 @@
       <mu2>0.2</mu2>
     </gazebo>
-    <gazebo reference="base_footprint">
+    <gazebo reference="$(arg base_frame_id)">
       <mu1>0.2</mu1>
       <mu2>0.2</mu2>
