Commit message: Removed all references to the realsense cameras. Removed unecessary code. Changed default values of arguments in launcher files. Opted for a "Generate-Then-Use" approach when changing the nav2 yaml file parameters for better debugging.

File: vizzy_description/robots/vizzy.urdf.xacro (robot description, xacro)
@@ -14,6 +14,4 @@
   <!-- Disable laser sensors -->
   <xacro:arg name="disable_laser" default="true"/>
-  <!-- Disable depth camera -->
-  <xacro:arg name="disable_3d_sensor" default="true"/>
   <!-- Includes -->
   <!-- Misc common stuff such as constant definitions -->
@@ -22,6 +20,4 @@
   <!-- Hokuyo URG-04LX laser scanner -->
   <xacro:include filename="$(find vizzy_description)/urdf/sensors/hokuyo_04lx_laser.urdf.xacro"/>
-  <!-- RealSense D435 -->
-  <xacro:include filename="$(find vizzy_description)/urdf/sensors/_d435.urdf.xacro"/>
   <!-- Robot body -->
   <!-- Base -->
@@ -74,10 +70,4 @@
     </xacro:hokuyo_04lx_laser>
   </xacro:unless>
-  <!-- Instantiate depth camera -->
-  <xacro:unless value="$(arg disable_3d_sensor)">
-    <xacro:sensor_d435 name="realsense" parent="waist_link">
-      <origin xyz="-0.09516 0.143 0.0" rpy="${-M_PI/2} ${M_PI} 0"/> <!-- In the drawing z=0.158!!!-->
-    </xacro:sensor_d435>
-  </xacro:unless>
   <!-- Instantiate plugins common to ROS and Yarp -->
   <xacro:joint_state_publisher/>
@@ -85,11 +75,4 @@
   <xacro:camera_plugin name="l_camera" prefix="l"/>
   <xacro:camera_plugin name="r_camera" prefix="r"/>
-  <!-- Instantiate Yarp plugins -->
-  <xacro:if value="$(arg use_yarp)">
-    <xacro:torso_gazebo_control/>
-    <xacro:head_gazebo_control/>
-    <xacro:left_arm_gazebo_control/>
-    <xacro:right_arm_gazebo_control/>
-  </xacro:if>
   <!-- Instantiate ROS plugins -->
   <xacro:unless value="$(arg use_yarp)">

Commit message: Basic Navigation Completed (#5)
* Adding necessary code for real robot navigation. Removed unecessary code from env_loader.sh. Corrected bug in navigation_launch.py: "use_sim_time" variable was not being used.

* Removed unecessary code. Created new python launcher for URDF creation and state publishers deployment.

* Updated CMakeLists.txt files and package.xml files to include the new code implemented for use in the real robot.

* Corrected segway_rmp_ros2 package name in package.xml of vizzy_robot.

* Removed unecessary code.

* Added comments detailing more about the transition from ROS1 to ROS2. Corrected substitution related to transition in file vizzy_real_launch.xml. Removed unecessary code.

* Refactored the code to remove the usage of the "machine" attribute from ROS1 (unsupported in ROS2).

* Removed obstacle map usage for now.

* Corrected file name.

* Corrected file package name.

* Corrected package name regarding auxiliary_vizzy_launch.py.

* Corrected variable substitution with LaunchConfiguration in auxiliary_vizzy_launch.py launcher.

* Removed unecessary code.

* Passed variable to auxiliary_vizzy_launch for testing.

* Inserted remaining variables in launch of auxiliary_vizzy_launch.py.

* Harcoded "use_sim_time" parameter in auxiliary_vizzy_launcher.py.

* Added joint_state_publisher and robot_state_publisher dependencies.

* Removed joint_state_publisher and robot_state_publisher from package.xml and CMakeLists.txt.

* Corrected executable name from segway_rmp_ros2_node to segway_rmp_node_ros2.

* Removed docking-specific code.

* Removed unecessary code.

* Changed executable name from urg_node to urg_node_driver.

* Added vizzy_sensors package.

* Corrected bug in transition from ROS1 to ROS2: forgot to replace catkin by ament_cmake.

* Removed unecessary code.

* Removed unecessary code.

* Removed unecessary code.

* Added necessary code and refactored CMakeLists.txt for package vizzy_sensors.

* Added necessary code.

* Removed unecessary code.

* Removed unecessary code.

* Removed unecessary code.

* Removed unecessary code.

* Refactored headers to ROS2 format.

* Refactored CPP code from ROS1 to ROS2.

* Refactored CPP code to work with ROS2.

* Refactored nan_to_inf_filter.h for ROS2 and higher efficiency.

* Refactored the ScanAngleFilter node to work with ROS2.

* Trying to fix node declaration issues in scan_angle_filter.h.

* Corrected code for compiler error-free ROS2 build.

* Corrected hokuyo laser filter ROS2 parameters.

* Refactored Hokuyo configurations to work with ROS2. Removed unecessary code.

* Added explicit "odometry" frame id in the segway_rmp_ros2 launch.

* Adjusted scan topic names. Corrected code to import the correct map file.

* Corrected syntax in vizzy_real_launch.xml "if" conditions.

* Corrected topic names mismatches in nav2_configuration_real.yaml. Inserted rear scan usage into AMCL.

* Found and corrected bug: navigation stack was using the topic /nav_hokuyo/front/scan instead of /scan.

* Trying to fix bug of incorrect frame_id name published with the laser scans.

* Corrected typo.

* Corrected laser frame id names and parameter name for the urg_node.

* Corrected the parameter name to correctly apply the map yaml file from "map_file" to "map_yaml". Changed the default value for "use_obstacles" to true.

* Trying to correctly pass on the parameters of the scan topics to AMCL.

* Corrected parameter name in AMCL configuration. No multiple scan topics are allowed.

* Added ROS_MASTER export in env loader.

* Corrected nav2 parameters related to topic names.

* Added frame_id parameter to segway_rmp_ros2 node.

* Adding logs to laser scan footprint filter.

* Added include for the launcher of the laser filters.

* Changed nav2 parameters for a greater min_range.

* Changed 4cm min range from raytrace to obstacle in nav2 configurations.

* Removed need for filtered scans through C++ code and removed unecessary code.

* Created all the parent variables necessary for the main launch file to have configurable parameters to control the entire launch stack of the real Vizzy. Removed necessity of second Nav2 configuration file (simulated and real Vizzy now use the same YAML with parameter substitutions). Cleaned code.

* Removed all references to the realsense cameras. Removed unecessary code. Changed default values of arguments in launcher files. Opted for a "Generate-Then-Use" approach when changing the nav2 yaml file parameters for better debugging.

* Testing input arguments for simulation launch. Corrected for arguments that were not well propagated.

* Corrected pose parameter propagation in simulation launch and removed unecessary code.

* Corrected variable declaration and propagation bugs.

* Adding new solo footprint filter.

* Corrected parameter propagation for filter launcher.

* Added more configurable parameters for debugging.

* Added string to boolean conversion in parameter file.

* Converted the necessary parameters to floats in the parameter file.

* Added parameter for usage without the navigation stack in the real robot and paramteres for beam skipping in AMCL usage.

* Corrected conversion from string to boolean in navigation stack launch.

* Added linear_odom_scale and angular_odom_scale to segway driver parameters.

* Corrected default values for segway drivers parameters.

* Changed default value for log level to 'info'.

* Adjusted nav2 parameters.

* Changed nav2 parameter values.

* Changed nav2 parameter values.

* Changed default values of nav2 parameters. Added configurable parameter on launch: controller_frequency.

* Added configurable parameters to simulation launch and changed default values for Nav2 parameters.

* Changed robot radius default value in Nav2 costmaps configurations paramters.

* Changed default value for global costmap update frequency.

* Changed default values of Nav2 parameters. Inserting support for RPP and MPPI controllers as well as the already supported DWB controller. Changed package files to insert new controllers as dependencies.

* Finished developing functionality of user choosing the controller plugin to use between DWB, RPP and MPPI, both in simulation and reality usage. When choosing DWB, the user can still configure all of the previous configurable parameters.

* Changed default value for planner server and made it configurable on startup.

* Changed default values and changed planner frequency in custom BT XML.

* Made the global planner frequency configurable on launch for the BT XML file.

* Changed default values for angular velocities and acceleration mppi controller.

* Changed mppi controller wz_max for testing purposes.

* Changed default wz_std value.

* Added Theta* Global Planner plugin support. User can now choose which Global Planner plugin to use. Changed Nav2 parameters' default values.

* Made the 'robot_radius' local and global costmap parameters configurable.

* Added smoother to custom BT XML file.

* Made some nav2 parameters configurable for the user.

* Added more configurable parameters by the user to Nav2 configurations.

* Changed default nav2 values to tested ones.

* Updated custom RViz configuration file to show more topics in simulation startup.

* Removed useless parameters in Nav2 configuration and added wz_std as a configurable parameter by the user.

* Added comments to the custom BT XML file. Updated custom RViz configuration file. Simplified launch arguments descriptions in navigation stack launch.

* Added dynamic controller change based on environment constraints.

* Added explicit min and max obstacle height parameters for local costmap to function in simulation.

* Updated logs and comments.

* Changed default parameters to test in real Vizzy.

* Added system dependency (xterm) to package.xml file.

* Refactored BT XML file for better dynamic handling of controller change. Changed some comments. Adapted configurable parameters for new dynamic system.

* Added necessary parameters to global planner to update obstacles in costmap.

* Changed Smoother Server plugin to use contrained_smoother. Added configurable parameter in Velocity Smoother Server.

* Changed default value for velocity smoother feedback type.

* Added maps to the vizzy_navigation package.

* Corrected map yaml files and removed unecessary maps.

* Add sections for vizzy_robot and vizzy_sensors in README

---------

Co-authored-by: João Duarte Penha Lopes <JPLDevMaster>

File: vizzy_description/robots/vizzy.urdf.xacro (robot description, xacro)
@@ -6,14 +6,11 @@
 -->
 <robot  name="vizzy" xmlns:xacro="http://ros.org/wiki/xacro" >
-  <!-- Load Yarp plugins for real robot execution -->
   <xacro:arg name="use_yarp" default="false"/>
-  <!-- Load full inertial and collision model or a simplified model -->
   <xacro:arg name="use_full_gazebo_model" default="false"/>
-  <!-- Load a fully detailed hand model with properly modeled links and joints -->
   <xacro:arg name="use_full_hand_model" default="false"/>
-  <!-- Disable laser sensors -->
-  <xacro:arg name="disable_laser" default="true"/>
-  <!-- Disable depth camera -->
-  <xacro:arg name="disable_3d_sensor" default="true"/>
+  <xacro:arg name="disable_laser" default="false"/>
+  <xacro:arg name="odom_topic"         default="/odom" />
+  <xacro:arg name="odom_frame_id"      default="odometry" />
+  <xacro:arg name="base_frame_id"   default="base_footprint" />
   <!-- Includes -->
   <!-- Misc common stuff such as constant definitions -->
@@ -22,6 +19,4 @@
   <!-- Hokuyo URG-04LX laser scanner -->
   <xacro:include filename="$(find vizzy_description)/urdf/sensors/hokuyo_04lx_laser.urdf.xacro"/>
-  <!-- RealSense D435 -->
-  <xacro:include filename="$(find vizzy_description)/urdf/sensors/_d435.urdf.xacro"/>
   <!-- Robot body -->
   <!-- Base -->
@@ -74,10 +69,4 @@
     </xacro:hokuyo_04lx_laser>
   </xacro:unless>
-  <!-- Instantiate depth camera -->
-  <xacro:unless value="$(arg disable_3d_sensor)">
-    <xacro:sensor_d435 name="realsense" parent="waist_link">
-      <origin xyz="-0.09516 0.143 0.0" rpy="${-M_PI/2} ${M_PI} 0"/> <!-- In the drawing z=0.158!!!-->
-    </xacro:sensor_d435>
-  </xacro:unless>
   <!-- Instantiate plugins common to ROS and Yarp -->
   <xacro:joint_state_publisher/>
@@ -85,11 +74,4 @@
   <xacro:camera_plugin name="l_camera" prefix="l"/>
   <xacro:camera_plugin name="r_camera" prefix="r"/>
-  <!-- Instantiate Yarp plugins -->
-  <xacro:if value="$(arg use_yarp)">
-    <xacro:torso_gazebo_control/>
-    <xacro:head_gazebo_control/>
-    <xacro:left_arm_gazebo_control/>
-    <xacro:right_arm_gazebo_control/>
-  </xacro:if>
   <!-- Instantiate ROS plugins -->
   <xacro:unless value="$(arg use_yarp)">
